File: servo_shield.kicad_pcb (KiCad board)
At the start: 2 copper layers, 70 x 59 mm, 94 parts, among them J1 BARREL_JACK, J10 CONN_01X03, J11 CONN_01X02, J12 CONN_01X03, J13 CONN_01X03, J14 CONN_01X03, J2 NUNCHUCK_CONN, J3 CONN_02X19, J5 CONN_02X19, J6 CONN_01X03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

Commit message: Revision 2
Parts:
- added ?: , servo_shield:VIA_0.35mm_0.55mm, F.Cu at (192.7, 103.0)
- added ?: , servo_shield:VIA_0.35mm_0.55mm, F.Cu at (155.5, 93.8)
- moved ? 1.52 mm to (157.5, 89.8)
Connections:
- J11 pad 1: /BAT_GND -> /VIN
- J11 pad 2: GND -> /BAT_GND
- J2 pad 3: (no net) -> Net-(J2-Pad3)
- J2 pad 4: (no net) -> Net-(J2-Pad4)
- J3 pad 10: (no net) -> Net-(J3-Pad10)
- J3 pad 11: (no net) -> Net-(J3-Pad11)
- J3 pad 12: (no net) -> Net-(J3-Pad12)
- J3 pad 13: (no net) -> Net-(J3-Pad13)
- J3 pad 14: (no net) -> Net-(J3-Pad14)
- J3 pad 15: (no net) -> Net-(J3-Pad15)
- J3 pad 16: (no net) -> Net-(J3-Pad16)
- J3 pad 17: (no net) -> Net-(J3-Pad17)
- J3 pad 18: (no net) -> Net-(J3-Pad18)
- J3 pad 21: (no net) -> Net-(J3-Pad21)
- J3 pad 23: (no net) -> Net-(J3-Pad23)
- J3 pad 24: (no net) -> Net-(J3-Pad24)
- J3 pad 25: (no net) -> Net-(J3-Pad25)
- J3 pad 26: (no net) -> Net-(J3-Pad26)
- J3 pad 27: (no net) -> Net-(J3-Pad27)
- J3 pad 28: (no net) -> /POW_EN
- J3 pad 29: (no net) -> Net-(J3-Pad29)
- J3 pad 30: (no net) -> Net-(J3-Pad30)
- J3 pad 31: (no net) -> Net-(J3-Pad31)
- J3 pad 32: /POW_EN -> Net-(J3-Pad32)
- J3 pad 33: (no net) -> Net-(J3-Pad33)
- J3 pad 34: (no net) -> Net-(J3-Pad34)
- J3 pad 35: (no net) -> Net-(J3-Pad35)
- J3 pad 37: (no net) -> Net-(J3-Pad37)
- J3 pad 4: (no net) -> Net-(J3-Pad4)
- J3 pad 5: (no net) -> Net-(J3-Pad5)
- J3 pad 7: (no net) -> Net-(J3-Pad7)
- J3 pad 9: (no net) -> Net-(J3-Pad9)
- J5 pad 1: (no net) -> Net-(J5-Pad1)
- J5 pad 10: (no net) -> Net-(J5-Pad10)
- J5 pad 11: (no net) -> Net-(J5-Pad11)
- J5 pad 12: (no net) -> Net-(J5-Pad12)
- J5 pad 14: (no net) -> /PA_11
- J5 pad 16: (no net) -> Net-(J5-Pad16)
- J5 pad 17: (no net) -> Net-(J5-Pad17)
- J5 pad 18: /PB_11 -> Net-(J5-Pad18)
- J5 pad 19: (no net) -> Net-(J5-Pad19)
- J5 pad 21: (no net) -> Net-(J5-Pad21)
- J5 pad 22: (no net) -> Net-(J5-Pad22)
- J5 pad 23: (no net) -> /PA_8
- J5 pad 24: /PB_1 -> Net-(J5-Pad24)
- J5 pad 25: /PB_10 -> Net-(J5-Pad25)
- J5 pad 26: (no net) -> Net-(J5-Pad26)
- J5 pad 27: (no net) -> Net-(J5-Pad27)
- J5 pad 28: (no net) -> /PB_14
- J5 pad 29: (no net) -> Net-(J5-Pad29)
- J5 pad 3: (no net) -> Net-(J5-Pad3)
- J5 pad 30: (no net) -> Net-(J5-Pad30)
- J5 pad 31: /PB_3 -> Net-(J5-Pad31)
- J5 pad 33: (no net) -> /PA_10
- J5 pad 34: (no net) -> Net-(J5-Pad34)
- J5 pad 35: (no net) -> Net-(J5-Pad35)
- J5 pad 36: (no net) -> Net-(J5-Pad36)
- J5 pad 37: (no net) -> Net-(J5-Pad37)
- J5 pad 38: (no net) -> Net-(J5-Pad38)
- J5 pad 5: (no net) -> Net-(J5-Pad5)
- J5 pad 6: (no net) -> Net-(J5-Pad6)
- J5 pad 7: (no net) -> Net-(J5-Pad7)
- J5 pad 8: (no net) -> Net-(J5-Pad8)
- Q5 pad 1: /PB_11 -> /PA_11
- Q6 pad 1: /PB_1 -> /PB_14
- Q7 pad 1: /PB_10 -> /PA_8
- Q8 pad 1: /PB_3 -> /PA_10
Routing:
- net /PB_14: track 0.00 -> 21.2 mm
- net /PB_1: track 20.1 -> 0.00 mm
- net /PA_10: track 0.00 -> 17.9 mm
- net /PB_3: track 15.4 -> 0.00 mm
- net /PA_11: track 0.00 -> 11.8 mm
- net /PB_11: track 9.61 -> 0.00 mm
- net /VIN: track 54.2 -> 62.5 mm
- net /PA_8: track 0.00 -> 8.13 mm
- net /PB_10: track 6.70 -> 0.00 mm
- net Net-(J5-Pad24): track 0.00 -> 3.44 mm
- net /POW_EN: track 40.8 -> 43.0 mm
- net /BAT_GND: track 61.6 -> 60.5 mm
- net +3V3: track 40.7 -> 40.8 mm, vias 2 -> 1
Other:
- outline, holes or cut-outs redrawn
- board text added: "+3.3V"
- board text added: "2 x GND"
- board text added: "BAT GND"
- board text added: "Rev 2 May 28 2018"
- board text added: "VIN"
- board text removed: "Left to right: A6 A7 B11 B1 B10 B3"
- board text removed: "Rev 1 April 4 2018"
